File: hardware/devices/test-device/kicad/common.sch (KiCad schematic (older format))
At the start: 4 parts, among them J6 CONN_01X02

Commit message: board fixes
Parts:
- C1: footprint Capacitors_SMD:C_0603_HandSoldering -> Capacitors_SMD:C_1206
Changed lines of the file:
@@
 F 0 "C1" H 1775 2300 50  0000 L CNN
 F 1 "C" H 1775 2100 50  0000 L CNN
-F 2 "Capacitors_SMD:C_0603_HandSoldering" H 1788 2050 50  0001 C CNN
+F 2 "Capacitors_SMD:C_1206" H 1788 2050 50  0001 C CNN
 F 3 "" H 1750 2200 50  0001 C CNN
 	1    1750 2200
