File: hardware/devices/test-device/kicad/rj12.sch (KiCad schematic (older format))
At the start: 1 part, among them J5 RJ12

Commit message: board fixes
Parts:
- J5: footprint conn-rj11:molex_95501-2641 -> rj12:molex_95501-2641
Changed lines of the file:
@@
 F 0 "J5" H 2300 2450 50  0000 C CNN
 F 1 "RJ12" H 1950 2450 50  0000 C CNN
-F 2 "conn-rj11:molex_95501-2641" H 2100 1950 50  0001 C CNN
+F 2 "rj12:molex_95501-2641" H 2100 1950 50  0001 C CNN
 F 3 "" H 2100 1950 50  0001 C CNN
 	1    2100 1950
