File: hardware/devices/test-device/kicad/test-device.kicad_pcb (KiCad board)
At the start: 2 copper layers, 13 parts, among them J1 CONN_01X02, J2 CONN_01X02, J3 CONN_02X04, J4 CONN_01X02, J5 RJ12, J6 CONN_01X02, U1 STM32F030F4Px, U2 LD1117S33TR

Commit message: board fixes
Parts:
- J5: footprint conn-rj11:molex_95501-2641 -> rj12:molex_95501-2641
- moved J6 6.74 mm to (165.2, 101.4), turned to 0 degrees
- moved J2 5.86 mm to (160.1, 101.3), turned to 270 degrees
- moved C1 5.56 mm to (160.2, 104.6)
- moved R2 4.63 mm to (167.7, 102.6), turned to 90 degrees
- moved C3 4.61 mm to (163.7, 95.6)
- moved U1 4.37 mm to (168.7, 95.6)
- moved R1 2.77 mm to (162.7, 100.0), turned to 90 degrees
Routing:
- net /Power/GND: track 86.0 -> 115.4 mm
- net /common uc/BOOT0: track 7.23 -> 0.00 mm
- net Net-(J3-Pad5): track 16.2 -> 10.3 mm
- net Net-(J3-Pad4): track 25.8 -> 20.5 mm
- net Net-(J3-Pad7): track 12.6 -> 7.51 mm
- net Net-(J3-Pad8): track 16.1 -> 11.6 mm
- net /common uc/IN_3.3V: track 41.2 -> 45.5 mm
- net Net-(J3-Pad1): track 13.6 -> 9.34 mm
- net /RJ-12/TX: track 10.4 -> 6.07 mm
- net Net-(J3-Pad6): track 21.6 -> 17.7 mm
- net /RJ-12/INT: track 10.2 -> 6.68 mm
- net /RJ-12/RDY: track 12.6 -> 10.1 mm
- net /RJ-12/RX: track 12.9 -> 10.7 mm
- net Net-(J3-Pad3): track 11.2 -> 9.20 mm
- net /Power/IN_5V: track 22.2 -> 24.1 mm
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Other:
- board outline added: 29.8 x 25.8 mm
